File: 0603 display board/0603 display board.kicad_sch (KiCad schematic)
At the start: 58 parts

Commit message: finished first layout
Parts:
- D1, D10, D11, D12, D13, D14, D15, D16, D17, D18, D19, D2, D20, D21, D22, D23, D24, D25, D26, D27, D28, D29, D3, D30, D31, D32, D33, D34, D35, D36, D37, D38, D39, D4, D40, D41, D42, D43, D44, D45, D46, D47, D48, D49, D5, D50, D51, D52, D53, D54, D55, D56, D6, D7, D8, D9: renamed from D?; footprint (none) -> LED_SMD:LED_0603_1608Metric
- J1, J2: renamed from J?; footprint (none) -> Connector_PinHeader_2.54mm:PinHeader_1x14_P2.54mm_Vertical
Connections:
- net Cathode 1: no longer D1.2 (A), D2.2 (A), D3.2 (A), D4.2 (A), D5.2 (A), D6.2 (A), D7.2 (A), J2.13 (Pin_13)
- net Cathode 2: no longer D15.2 (A), D16.2 (A), D17.2 (A), D18.2 (A), D19.2 (A), D20.2 (A), D21.2 (A), J2.11 (Pin_11)
- net Cathode 3: no longer D27.2 (A), D28.2 (A), D29.2 (A), D30.2 (A), D31.2 (A), D34.2 (A), D35.2 (A), J2.9 (Pin_9)
- net Cathode 4: no longer D36.2 (A), D37.2 (A), D45.2 (A), D46.2 (A), D47.2 (A), D48.2 (A), D49.2 (A), J2.8 (Pin_8)
- net Cathode 5: no longer D50.2 (A), D51.2 (A), D52.2 (A), D53.2 (A), D54.2 (A), D55.2 (A), D56.2 (A), J2.7 (Pin_7)
- net Cathode 6: no longer D10.2 (A), D11.2 (A), D12.2 (A), D13.2 (A), D14.2 (A), D8.2 (A), D9.2 (A), J2.5 (Pin_5)
- net Cathode 7: no longer D22.2 (A), D23.2 (A), D24.2 (A), D25.2 (A), D26.2 (A), D32.2 (A), D33.2 (A), J2.3 (Pin_3)
- new net Digit 1: D1.2 (A), D2.2 (A), D3.2 (A), D4.2 (A), D5.2 (A), D6.2 (A), D7.2 (A), J2.13 (Pin_13)
- new net Digit 2: D15.2 (A), D16.2 (A), D17.2 (A), D18.2 (A), D19.2 (A), D20.2 (A), D21.2 (A), J2.11 (Pin_11)
- new net Digit 3: D27.2 (A), D28.2 (A), D29.2 (A), D30.2 (A), D31.2 (A), D34.2 (A), D35.2 (A), J2.9 (Pin_9)
- new net Digit 4: D36.2 (A), D37.2 (A), D45.2 (A), D46.2 (A), D47.2 (A), D48.2 (A), D49.2 (A), J2.8 (Pin_8)
- new net Digit 5: D50.2 (A), D51.2 (A), D52.2 (A), D53.2 (A), D54.2 (A), D55.2 (A), D56.2 (A), J2.7 (Pin_7)
- new net Digit 6: D10.2 (A), D11.2 (A), D12.2 (A), D13.2 (A), D14.2 (A), D8.2 (A), D9.2 (A), J2.5 (Pin_5)
- new net Digit 7: D22.2 (A), D23.2 (A), D24.2 (A), D25.2 (A), D26.2 (A), D32.2 (A), D33.2 (A), J2.3 (Pin_3)

Commit message: smaller footprint
Parts:
- D1, D10, D11, D12, D13, D14, D15, D16, D17, D18, D19, D2, D20, D21, D22, D23, D24, D25, D26, D27, D28, D29, D3, D30, D31, D32, D33, D34, D35, D36, D37, D38, D39, D4, D40, D41, D42, D43, D44, D45, D46, D47, D48, D49, D5, D50, D51, D52, D53, D54, D55, D56, D6, D7, D8, D9: footprint LED_SMD:LED_0603_1608Metric -> Evan's misc parts:LED_0603_smallpads
